Commit message: tipping_monitor , factorized default dimensions

File: rosmip/rosmip_description/urdf/rosmip_1.urdf.xacro (robot description, xacro)
@@ -1,19 +1,5 @@
 <?xml version="1.0"?>
 <robot name="rosmip_1" xmlns:xacro="http://www.ros.org/wiki/xacro">
-  <xacro:property name="chassis_length" value="0.035" />
-  <xacro:property name="chassis_width"  value="0.062" />
-  <xacro:property name="chassis_height" value="0.12" />
-  <xacro:property name="chassis_mass"   value="0.18" />
-  <xacro:property name="chassis_vert_offset" value="0.055" />
-  <xacro:property name="left_wheel_radius"  value="0.03" />
-  <xacro:property name="right_wheel_radius" value="0.03" />
-  <xacro:property name="wheel_width"  value="0.01" />
-  <xacro:property name="wheel_track"  value="0.083" />
-  <xacro:property name="wheel_mass"   value="0.01" />
-  <xacro:property name="wheel_joint_damping" value="0.01" />
-  <xacro:property name="wheel_joint_friction" value="0.01" />
-  <xacro:property name="high_definition_wheel_visual" value="true" />
-  <xacro:property name="high_definition_body_visual" value="true" />
-  <xacro:property name="use_infrared_marker" value="false" />
+  <xacro:include filename="$(find rosmip_description)/urdf/rosmip_defaults.urdf.xacro" />
   <xacro:include filename="$(find rosmip_description)/urdf/rosmip.urdf.xacro" />
 </robot>

File: rosmip/rosmip_description/urdf/rosmip_2.urdf.xacro (robot description, xacro)
@@ -1,18 +1,7 @@
 <?xml version="1.0"?>
 <robot name="rosmip_1" xmlns:xacro="http://www.ros.org/wiki/xacro">
-  <xacro:property name="chassis_length" value="0.035" />
-  <xacro:property name="chassis_width"  value="0.062" />
-  <xacro:property name="chassis_height" value="0.12" />
-  <xacro:property name="chassis_mass"   value="0.18" />
-  <xacro:property name="chassis_vert_offset" value="0.055" />
-  <xacro:property name="left_wheel_radius"  value="0.04" />
-  <xacro:property name="right_wheel_radius" value="0.04" />
-  <xacro:property name="wheel_width"  value="0.01" />
-  <xacro:property name="wheel_track"  value="0.083" />
-  <xacro:property name="wheel_mass"   value="0.01" />
-  <xacro:property name="wheel_joint_damping" value="0.01" />
-  <xacro:property name="wheel_joint_friction" value="0.01" />
-  <xacro:property name="high_definition_wheel_visual" value="true" />
-  <xacro:property name="high_definition_body_visual" value="false" />
+  <xacro:include filename="$(find rosmip_description)/urdf/rosmip_defaults.urdf.xacro" />
+  <xacro:property name="left_wheel_radius"  value="0.045" />
+  <xacro:property name="right_wheel_radius" value="0.045" />
   <xacro:property name="use_infrared_marker" value="true" />
   <xacro:include filename="$(find rosmip_description)/urdf/rosmip.urdf.xacro" />

File: rosmip/rosmip_description/urdf/rosmip_3.urdf.xacro (robot description, xacro)
@@ -2,19 +2,7 @@
 <!-- let's try a robot with different radius wheels -->
 <robot name="rosmip_3" xmlns:xacro="http://www.ros.org/wiki/xacro">
-  <xacro:property name="chassis_length" value="0.035" />
-  <xacro:property name="chassis_width"  value="0.062" />
-  <xacro:property name="chassis_height" value="0.12" />
-  <xacro:property name="chassis_mass"   value="0.18" />
-  <xacro:property name="chassis_vert_offset" value="0.055" />
-  <xacro:property name="left_wheel_radius"  value="0.0375" />
-  <xacro:property name="right_wheel_radius" value="0.0425" />
-  <xacro:property name="wheel_width"  value="0.01" />
-  <xacro:property name="wheel_track"  value="0.083" />
-  <xacro:property name="wheel_mass"   value="0.01" />
-  <xacro:property name="wheel_joint_damping" value="0.01" />
-  <xacro:property name="wheel_joint_friction" value="0.01" />
-  <xacro:property name="high_definition_wheel_visual" value="true" />
-  <xacro:property name="high_definition_body_visual" value="false" />
-  <xacro:property name="use_infrared_marker" value="true" />
+  <xacro:include filename="$(find rosmip_description)/urdf/rosmip_defaults.urdf.xacro" />
+  <xacro:property name="left_wheel_radius"  value="0.031" />
+  <xacro:property name="right_wheel_radius" value="0.029" />
   <xacro:include filename="$(find rosmip_description)/urdf/rosmip.urdf.xacro" />
 </robot>
