Commit message: bla

File: rosmip/rosmip_description/urdf/rosmip.urdf.xacro (robot description, xacro)
@@ -6,14 +6,14 @@
   <xacro:property name="chassis_width"  value="0.065" />
   <xacro:property name="chassis_height" value="0.12" />
-  <xacro:property name="chassis_mass"   value="0.2" />
-  <xacro:property name="chassis_vert_offset" value="0.1" /> <!-- 0.1-->
-  <xacro:property name="wheel_radius" value="0.045" />
+  <xacro:property name="chassis_mass"   value="0.18" />
+  <xacro:property name="chassis_vert_offset" value="0.085" /> <!-- 0.1-->
+  <xacro:property name="wheel_radius" value="0.03" />
   <xacro:property name="wheel_width"  value="0.01" />
   <xacro:property name="wheel_track"  value="0.08" />
-  <xacro:property name="wheel_mass"   value="0.02" />
+  <xacro:property name="wheel_mass"   value="0.01" />
   <!--<xacro:property name="wheel_joint_damping" value="0.2" />
   <xacro:property name="wheel_joint_friction" value="0.7" /> -->
   <xacro:property name="wheel_joint_damping" value="0.01" />
-  <xacro:property name="wheel_joint_friction" value="0.0" />
+  <xacro:property name="wheel_joint_friction" value="0.01" />
   <material name="light_grey"><color rgba="0.4 0.4 0.4 1.0" /></material>
   <material name="yellow"><color rgba="0.8 0.8 0.0 1.0" /></material>
@@ -34,5 +34,6 @@
 	<origin xyz="0 0 0" rpy="0 0 ${lr_reflect*PI/2}"/>
         <geometry>
-	  <mesh filename="package://rosmip_description/meshes/wheel_test.dae"/>
+	   <!--<mesh filename="package://rosmip_description/meshes/wheel_test.dae"/>-->
+	   <mesh filename="package://rosmip_description/meshes/wheel_60.dae"/>
         </geometry>
       </visual>
@@ -58,4 +59,5 @@
       <axis xyz="0 1 0" />
       <dynamics damping="${wheel_joint_damping}" friction="${wheel_joint_friction}"/>
+      <limit effort="1" velocity="10"/>
     </joint>
     <transmission name="${prefix}_wheel_trans">

Commit message: this time, i added the right files. fuck you git

File: rosmip/rosmip_description/urdf/rosmip.urdf.xacro (robot description, xacro)
@@ -10,10 +10,11 @@
   <xacro:property name="wheel_radius" value="0.03" />
   <xacro:property name="wheel_width"  value="0.01" />
-  <xacro:property name="wheel_track"  value="0.08" />
+  <xacro:property name="wheel_track"  value="0.083" />
   <xacro:property name="wheel_mass"   value="0.01" />
-  <!--<xacro:property name="wheel_joint_damping" value="0.2" />
-  <xacro:property name="wheel_joint_friction" value="0.7" /> -->
   <xacro:property name="wheel_joint_damping" value="0.01" />
   <xacro:property name="wheel_joint_friction" value="0.01" />
+  <!-- appearance -->
+  <xacro:property name="high_definition_wheel_visual" value="true" />
+  <xacro:property name="high_definition_body_visual" value="false" />
   <material name="light_grey"><color rgba="0.4 0.4 0.4 1.0" /></material>
   <material name="yellow"><color rgba="0.8 0.8 0.0 1.0" /></material>
@@ -25,16 +26,18 @@
     <link name="${prefix}_wheel_link">
       <visual>
-	<!--
-	<origin xyz="0 0 0" rpy="${PI/2} 0 0"/>
-        <geometry>
-	  <cylinder radius="${wheel_radius}" length="${wheel_width}"/>
-        </geometry>
-        <material name="yellow" />
-	-->
-	<origin xyz="0 0 0" rpy="0 0 ${lr_reflect*PI/2}"/>
-        <geometry>
-	   <!--<mesh filename="package://rosmip_description/meshes/wheel_test.dae"/>-->
-	   <mesh filename="package://rosmip_description/meshes/wheel_60.dae"/>
-        </geometry>
+	<xacro:unless value="${high_definition_wheel_visual}">
+	  <origin xyz="0 0 0" rpy="${PI/2} 0 0"/>
+          <geometry>
+	    <cylinder radius="${wheel_radius}" length="${wheel_width}"/>
+          </geometry>
+          <material name="yellow" />
+	</xacro:unless>
+	<xacro:if value="${high_definition_wheel_visual}">
+	  <origin xyz="0 0 0" rpy="0 0 ${lr_reflect*PI/2}"/>
+          <geometry>
+	    <!--<mesh filename="package://rosmip_description/meshes/wheel_test.dae"/>-->
+	    <mesh filename="package://rosmip_description/meshes/wheel_60.dae"/>
+          </geometry>
+	</xacro:if>
       </visual>
       <collision>
@@ -50,6 +53,4 @@
     <gazebo reference="${prefix}_wheel_link">
       <material>Gazebo/DarkGrey</material>
-      <!--<material>Gazebo/WoodFloor</material>-->
-      <!--<material>Gazebo/WoodPallet</material>-->
     </gazebo>
     <joint name="${prefix}_wheel_joint" type="continuous">
@@ -89,6 +90,10 @@
       <origin xyz="0 0 ${chassis_vert_offset}" rpy="0 0 0"/>
       <geometry>
-	<mesh filename="package://rosmip_description/meshes/body_minion.dae"/>
-	<!--<box size="${chassis_length} ${chassis_width} ${chassis_height}"/>-->
+	<xacro:if value="${high_definition_body_visual}">
+	  <mesh filename="package://rosmip_description/meshes/body_minion.dae"/>
+	</xacro:if>
+	<xacro:unless value="${high_definition_body_visual}">
+	  <box size="${chassis_length} ${chassis_width} ${chassis_height}"/>
+	</xacro:unless>
       </geometry>
       <!--<material name="yellow" />-->

Commit message: tweaked simulator dimensions

File: rosmip/rosmip_description/urdf/rosmip.urdf.xacro (robot description, xacro)
@@ -3,9 +3,9 @@
   <!-- Dimensions -->
   <xacro:property name="PI" value="3.1415926535897931" />
-  <xacro:property name="chassis_length" value="0.04" /> <!-- 0.005-->
-  <xacro:property name="chassis_width"  value="0.065" />
+  <xacro:property name="chassis_length" value="0.035" />
+  <xacro:property name="chassis_width"  value="0.062" />
   <xacro:property name="chassis_height" value="0.12" />
   <xacro:property name="chassis_mass"   value="0.18" />
-  <xacro:property name="chassis_vert_offset" value="0.085" /> <!-- 0.1-->
+  <xacro:property name="chassis_vert_offset" value="0.085" />
   <xacro:property name="wheel_radius" value="0.03" />
   <xacro:property name="wheel_width"  value="0.01" />
@@ -74,8 +74,8 @@
   </xacro:macro>
   <xacro:wheel prefix="left" lr_reflect="1">
-    <origin xyz="0 ${wheel_track/2} ${wheel_radius+0.0}" rpy="0 0 0" />
+    <origin xyz="0 ${(wheel_track-wheel_width)/2} ${wheel_radius}" rpy="0 0 0" />
   </xacro:wheel>
   <xacro:wheel prefix="right"  lr_reflect="-1">
-    <origin xyz="0 ${-wheel_track/2} ${wheel_radius+0.0}" rpy="0 0 0" />
+    <origin xyz="0 ${-(wheel_track-wheel_width)/2} ${wheel_radius}" rpy="0 0 0" />
   </xacro:wheel>
   <!-- Body -->

Commit message: initial support for mocap

File: rosmip/rosmip_description/urdf/rosmip.urdf.xacro (robot description, xacro)
@@ -20,4 +20,6 @@
   <material name="yellow"><color rgba="0.8 0.8 0.0 1.0" /></material>
   <material name="black"><color rgba="0.15 0.15 0.15 1.0" /></material>
+  <!-- infrared marker -->
+  <xacro:property name="use_infrared_marker" value="true" />
   <!-- Inertia macros -->
   <xacro:include filename="$(find rosmip_description)/urdf/inertias.urdf.xacro" />
@@ -89,13 +91,15 @@
     <visual>
       <origin xyz="0 0 ${chassis_vert_offset}" rpy="0 0 0"/>
-      <geometry>
 	<xacro:if value="${high_definition_body_visual}">
-	  <mesh filename="package://rosmip_description/meshes/body_minion.dae"/>
+	  <geometry>
+	    <mesh filename="package://rosmip_description/meshes/body_minion.dae"/>
+	  </geometry>
 	</xacro:if>
 	<xacro:unless value="${high_definition_body_visual}">
-	  <box size="${chassis_length} ${chassis_width} ${chassis_height}"/>
+	  <geometry>
+	    <box size="${chassis_length} ${chassis_width} ${chassis_height}"/>
+	  </geometry>
+	  <material name="yellow" />
 	</xacro:unless>
-      </geometry>
-      <!--<material name="yellow" />-->
     </visual>
     <collision>
@@ -114,4 +118,35 @@
   </gazebo>
   -->
+  <!-- Infrared Marker -->
+  <xacro:if value="${use_infrared_marker}">
+    <xacro:property name="irm_z" value="0.15" />
+    <xacro:property name="irm_dx" value="0.01" />
+    <xacro:property name="irm_dy" value="0.1" />
+    <xacro:property name="irm_dz" value="0.01" />
+    <xacro:property name="irm_mass" value="0.01" />
+    <link name="irm_link">
+      <visual>
+	<origin xyz="0 0 0" rpy="0 0 0"/>
+	<geometry>
+	  <!--<box size="${irm_dx} ${irm_dy} ${irm_dz}"/>-->
+	  <mesh filename="package://rosmip_description/meshes/ir_marker.dae"/>
+	</geometry>
+      </visual>
+      <collision>
+	<origin xyz="0 0 0" rpy="0 0 0"/>
+	<geometry>
+	  <box size="${irm_dx} ${irm_dy} ${irm_dz}"/>
+	</geometry>
+      </collision>
+      <xacro:inertial_cuboid_with_pose mass="${irm_mass}" x_length="${irm_dx}" y_length="${irm_dy}" z_length="${irm_dz}">
+	<origin xyz="0.00  0.00 0" rpy="0 0 0"/>
+      </xacro:inertial_cuboid_with_pose>
+    </link>
+    <joint name="irm_joint" type="fixed">
+      <origin xyz="0 0 ${irm_z}" rpy="0 0 0" />
+      <parent link="chassis_link"/>
+      <child link="irm_link" />
+    </joint>
+  </xacro:if>
   <!-- IMU -->
   <link name="imu_link"/>

Commit message: moved description of infrared marker to smocap package

File: rosmip/rosmip_description/urdf/rosmip.urdf.xacro (robot description, xacro)
@@ -120,27 +120,6 @@
   <!-- Infrared Marker -->
   <xacro:if value="${use_infrared_marker}">
+    <xacro:include filename="$(find smocap)/urdf/ir_marker.urdf.xacro" />
     <xacro:property name="irm_z" value="0.15" />
-    <xacro:property name="irm_dx" value="0.01" />
-    <xacro:property name="irm_dy" value="0.1" />
-    <xacro:property name="irm_dz" value="0.01" />
-    <xacro:property name="irm_mass" value="0.01" />
-    <link name="irm_link">
-      <visual>
-	<origin xyz="0 0 0" rpy="0 0 0"/>
-	<geometry>
-	  <!--<box size="${irm_dx} ${irm_dy} ${irm_dz}"/>-->
-	  <mesh filename="package://rosmip_description/meshes/ir_marker.dae"/>
-	</geometry>
-      </visual>
-      <collision>
-	<origin xyz="0 0 0" rpy="0 0 0"/>
-	<geometry>
-	  <box size="${irm_dx} ${irm_dy} ${irm_dz}"/>
-	</geometry>
-      </collision>
-      <xacro:inertial_cuboid_with_pose mass="${irm_mass}" x_length="${irm_dx}" y_length="${irm_dy}" z_length="${irm_dz}">
-	<origin xyz="0.00  0.00 0" rpy="0 0 0"/>
-      </xacro:inertial_cuboid_with_pose>
-    </link>
     <joint name="irm_joint" type="fixed">
       <origin xyz="0 0 ${irm_z}" rpy="0 0 0" />

Commit message: lots..., switching to gazebo 9

File: rosmip/rosmip_description/urdf/rosmip.urdf.xacro (robot description, xacro)
@@ -7,5 +7,5 @@
   <xacro:property name="chassis_height" value="0.12" />
   <xacro:property name="chassis_mass"   value="0.18" />
-  <xacro:property name="chassis_vert_offset" value="0.085" />
+  <xacro:property name="chassis_vert_offset" value="0.055" />
   <xacro:property name="wheel_radius" value="0.03" />
   <xacro:property name="wheel_width"  value="0.01" />
@@ -76,8 +76,8 @@
   </xacro:macro>
   <xacro:wheel prefix="left" lr_reflect="1">
-    <origin xyz="0 ${(wheel_track-wheel_width)/2} ${wheel_radius}" rpy="0 0 0" />
+    <origin xyz="0 ${(wheel_track-wheel_width)/2} 0" rpy="0 0 0" />
   </xacro:wheel>
   <xacro:wheel prefix="right"  lr_reflect="-1">
-    <origin xyz="0 ${-(wheel_track-wheel_width)/2} ${wheel_radius}" rpy="0 0 0" />
+    <origin xyz="0 ${-(wheel_track-wheel_width)/2} 0" rpy="0 0 0" />
   </xacro:wheel>
   <!-- Body -->
@@ -124,5 +124,5 @@
      <xacro:include filename="$(find smocap)/urdf/ir_marker.urdf.xacro" />
      <xacro:ir_marker root_link="$(arg root_link)" mesh="$(arg mesh)"/>
-    <xacro:property name="irm_z" value="0.15" />
+    <xacro:property name="irm_z" value="0.12" />
     <joint name="irm_joint" type="fixed">
       <origin xyz="0 0 ${irm_z}" rpy="0 0 0" />

Commit message: made per-robot dimensions and control configurations

File: rosmip/rosmip_description/urdf/rosmip.urdf.xacro (robot description, xacro)
@@ -3,17 +3,18 @@
   <!-- Dimensions -->
   <xacro:property name="PI" value="3.1415926535897931" />
-  <xacro:property name="chassis_length" value="0.035" />
-  <xacro:property name="chassis_width"  value="0.062" />
-  <xacro:property name="chassis_height" value="0.12" />
-  <xacro:property name="chassis_mass"   value="0.18" />
-  <xacro:property name="chassis_vert_offset" value="0.055" />
-  <xacro:property name="wheel_radius" value="0.03" />
-  <xacro:property name="wheel_width"  value="0.01" />
-  <xacro:property name="wheel_track"  value="0.083" />
-  <xacro:property name="wheel_mass"   value="0.01" />
-  <xacro:property name="wheel_joint_damping" value="0.01" />
-  <xacro:property name="wheel_joint_friction" value="0.01" />
+  <!-- <xacro:property name="chassis_length" value="0.035" /> -->
+  <!-- <xacro:property name="chassis_width"  value="0.062" /> -->
+  <!-- <xacro:property name="chassis_height" value="0.12" /> -->
+  <!-- <xacro:property name="chassis_mass"   value="0.18" /> -->
+  <!-- <xacro:property name="chassis_vert_offset" value="0.055" /> -->
+  <!-- <xacro:property name="wheel_radius" value="0.03" /> -->
+  <!-- <xacro:property name="wheel_width"  value="0.01" /> -->
+  <!-- <xacro:property name="wheel_track"  value="0.083" /> -->
+  <!-- <xacro:property name="wheel_mass"   value="0.01" /> -->
+  <!-- <xacro:property name="wheel_joint_damping" value="0.01" /> -->
+  <!-- <xacro:property name="wheel_joint_friction" value="0.01" /> -->
   <!-- appearance -->
-  <xacro:property name="high_definition_wheel_visual" value="true" />
+  <!-- <xacro:property name="high_definition_wheel_visual" value="true" /> -->
+  <xacro:property name="wheel_mesh_scale" value="${wheel_radius/0.03}" />
   <xacro:property name="high_definition_body_visual" value="false" />
   <material name="light_grey"><color rgba="0.4 0.4 0.4 1.0" /></material>
@@ -38,6 +39,5 @@
 	  <origin xyz="0 0 0" rpy="0 0 ${lr_reflect*PI/2}"/>
           <geometry>
-	    <!--<mesh filename="package://rosmip_description/meshes/wheel_test.dae"/>-->
-	    <mesh filename="package://rosmip_description/meshes/wheel_60.dae"/>
+	    <mesh scale="1. ${wheel_mesh_scale} ${wheel_mesh_scale}" filename="package://rosmip_description/meshes/wheel_60.dae"/>
           </geometry>
 	</xacro:if>

Commit message: fixed pure pursuit and move base simulations

File: rosmip/rosmip_description/urdf/rosmip.urdf.xacro (robot description, xacro)
@@ -16,5 +16,4 @@
   <!-- appearance -->
   <!-- <xacro:property name="high_definition_wheel_visual" value="true" /> -->
-  <xacro:property name="wheel_mesh_scale" value="${wheel_radius/0.03}" />
   <xacro:property name="high_definition_body_visual" value="false" />
   <material name="light_grey"><color rgba="0.4 0.4 0.4 1.0" /></material>
@@ -26,5 +25,6 @@
   <xacro:include filename="$(find rosmip_description)/urdf/inertias.urdf.xacro" />
   <!-- Wheels -->
-  <xacro:macro name="wheel" params="prefix lr_reflect *joint_pose">
+  <xacro:macro name="wheel" params="prefix wheel_radius lr_reflect *joint_pose">
+    <xacro:property name="wheel_mesh_scale" value="${wheel_radius/0.03}" />
     <link name="${prefix}_wheel_link">
       <visual>
@@ -75,8 +75,8 @@
     </transmission>
   </xacro:macro>
-  <xacro:wheel prefix="left" lr_reflect="1">
+  <xacro:wheel prefix="left" wheel_radius="${left_wheel_radius}" lr_reflect="1">
     <origin xyz="0 ${(wheel_track-wheel_width)/2} 0" rpy="0 0 0" />
   </xacro:wheel>
-  <xacro:wheel prefix="right"  lr_reflect="-1">
+  <xacro:wheel prefix="right"  wheel_radius="${right_wheel_radius}" lr_reflect="-1">
     <origin xyz="0 ${-(wheel_track-wheel_width)/2} 0" rpy="0 0 0" />
   </xacro:wheel>

File: rosmip/rosmip_description/urdf/rosmip_2.urdf.xacro (robot description, xacro)
@@ -6,5 +6,6 @@
   <xacro:property name="chassis_mass"   value="0.18" />
   <xacro:property name="chassis_vert_offset" value="0.055" />
-  <xacro:property name="wheel_radius" value="0.04" />
+  <xacro:property name="left_wheel_radius"  value="0.04" />
+  <xacro:property name="right_wheel_radius" value="0.04" />
   <xacro:property name="wheel_width"  value="0.01" />
   <xacro:property name="wheel_track"  value="0.083" />

File: rosmip/rosmip_description/urdf/rosmip_3.urdf.xacro (robot description, xacro)
@@ -1,4 +1,5 @@
 <?xml version="1.0"?>
-<robot name="rosmip_1" xmlns:xacro="http://www.ros.org/wiki/xacro">
+<!-- let's try a robot with different radius wheels -->
+<robot name="rosmip_3" xmlns:xacro="http://www.ros.org/wiki/xacro">
   <xacro:property name="chassis_length" value="0.035" />
   <xacro:property name="chassis_width"  value="0.062" />
@@ -6,6 +7,6 @@
   <xacro:property name="chassis_mass"   value="0.18" />
   <xacro:property name="chassis_vert_offset" value="0.055" />
-  <xacro:property name="left_wheel_radius"  value="0.03" />
-  <xacro:property name="right_wheel_radius" value="0.03" />
+  <xacro:property name="left_wheel_radius"  value="0.0375" />
+  <xacro:property name="right_wheel_radius" value="0.0425" />
   <xacro:property name="wheel_width"  value="0.01" />
   <xacro:property name="wheel_track"  value="0.083" />

Commit message: added aruco marker

File: rosmip/rosmip_description/urdf/rosmip.urdf.xacro (robot description, xacro)
@@ -16,10 +16,10 @@
   <!-- appearance -->
   <!-- <xacro:property name="high_definition_wheel_visual" value="true" /> -->
-  <xacro:property name="high_definition_body_visual" value="false" />
+  <!-- <xacro:property name="high_definition_body_visual" value="false" /> -->
   <material name="light_grey"><color rgba="0.4 0.4 0.4 1.0" /></material>
   <material name="yellow"><color rgba="0.8 0.8 0.0 1.0" /></material>
   <material name="black"><color rgba="0.15 0.15 0.15 1.0" /></material>
   <!-- infrared marker -->
-  <xacro:property name="use_infrared_marker" value="true" />
+  <!-- <xacro:property name="use_infrared_marker" value="true" /> -->
   <!-- Inertia macros -->
   <xacro:include filename="$(find rosmip_description)/urdf/inertias.urdf.xacro" />
@@ -90,11 +90,13 @@
   <link name="chassis_link">
     <visual>
-      <origin xyz="0 0 ${chassis_vert_offset}" rpy="0 0 0"/>
 	<xacro:if value="${high_definition_body_visual}">
+	  <origin xyz="0.009 0 ${chassis_vert_offset-0.025}" rpy="${pi/2} 0 ${pi/2}"/>
 	  <geometry>
-	    <mesh filename="package://rosmip_description/meshes/body_minion.dae"/>
+	    <!--<mesh filename="package://rosmip_description/meshes/body_minion.dae"/>-->
+	    <mesh filename="package://rosmip_description/meshes/body_murat.dae"/>
 	  </geometry>
 	</xacro:if>
 	<xacro:unless value="${high_definition_body_visual}">
+	  <origin xyz="0 0 ${chassis_vert_offset}" rpy="0 0 0"/>
 	  <geometry>
 	    <box size="${chassis_length} ${chassis_width} ${chassis_height}"/>
@@ -131,4 +133,20 @@
     </joint>
   </xacro:if>
+  <!-- Aruco Marker -->
+  <xacro:if value="${use_aruco_marker}">
+    <xacro:arg name="root_link" default="irm_link"/>
+    <xacro:arg name="marker_texture" default="Aruco14"/>
+    <xacro:include filename="$(find smocap)/urdf/chessboard.urdf.xacro" />
+    <xacro:property name="chsbrd_dx"   value="0.05" />
+    <xacro:property name="chsbrd_dy"   value="0.05" />
+    <xacro:property name="chsbrd_dz"   value="0.0025" />
+    <xacro:chessboard root_link="$(arg root_link)" texture="$(arg marker_texture)" static="false"/>
+    <xacro:property name="irm_z" value="0.098" />
+    <joint name="irm_joint" type="fixed">
+      <origin xyz="0.0025 0 ${irm_z}" rpy="0 0 0" />
+      <parent link="chassis_link"/>
+      <child link="irm_link" />
+    </joint>
+  </xacro:if>
   <!-- IMU -->
   <link name="imu_link"/>

File: rosmip/rosmip_description/urdf/rosmip_1.urdf.xacro (robot description, xacro)
@@ -14,4 +14,6 @@
   <xacro:property name="wheel_joint_friction" value="0.01" />
   <xacro:property name="high_definition_wheel_visual" value="true" />
+  <xacro:property name="high_definition_body_visual" value="true" />
+  <xacro:property name="use_infrared_marker" value="false" />
   <xacro:include filename="$(find rosmip_description)/urdf/rosmip.urdf.xacro" />
 </robot>

File: rosmip/rosmip_description/urdf/rosmip_2.urdf.xacro (robot description, xacro)
@@ -14,4 +14,6 @@
   <xacro:property name="wheel_joint_friction" value="0.01" />
   <xacro:property name="high_definition_wheel_visual" value="true" />
+  <xacro:property name="high_definition_body_visual" value="false" />
+  <xacro:property name="use_infrared_marker" value="true" />
   <xacro:include filename="$(find rosmip_description)/urdf/rosmip.urdf.xacro" />
 </robot>

File: rosmip/rosmip_description/urdf/rosmip_3.urdf.xacro (robot description, xacro)
@@ -15,4 +15,6 @@
   <xacro:property name="wheel_joint_friction" value="0.01" />
   <xacro:property name="high_definition_wheel_visual" value="true" />
+  <xacro:property name="high_definition_body_visual" value="false" />
+  <xacro:property name="use_infrared_marker" value="true" />
   <xacro:include filename="$(find rosmip_description)/urdf/rosmip.urdf.xacro" />
 </robot>
