Commit message: made send_tf changeable, added camera, record smocap

File: rosmip/rosmip_description/urdf/rosmip.urdf.xacro (robot description, xacro)
@@ -17,4 +17,5 @@
   <!-- <xacro:property name="high_definition_wheel_visual" value="true" /> -->
   <!-- <xacro:property name="high_definition_body_visual" value="false" /> -->
+  <xacro:include filename="$(find common_robots)/urdf/sensors.urdf.xacro" />
   <material name="light_grey"><color rgba="0.4 0.4 0.4 1.0" /></material>
   <material name="yellow"><color rgba="0.8 0.8 0.0 1.0" /></material>
@@ -94,5 +95,6 @@
 	  <geometry>
 	    <!--<mesh filename="package://rosmip_description/meshes/body_minion.dae"/>-->
-	    <mesh filename="package://rosmip_description/meshes/body_murat.dae"/>
+	    <!--<mesh filename="package://rosmip_description/meshes/body_murat.dae"/>-->
+	    <mesh filename="package://rosmip_description/meshes/rosmip_chassis.dae"/>
 	  </geometry>
 	</xacro:if>
@@ -156,4 +158,11 @@
     <child link="imu_link" />
   </joint>
+  <!-- Camera -->
+  <xacro:if value="${use_eachine_camera}">
+    <xacro:property name="cam_look_down_deg" value="0." />
+    <xacro:cs_camera_eachine>
+      <origin xyz="0.025 0 0.085" rpy="0 ${cam_look_down_deg/180*pi}} 0" />
+    </xacro:cs_camera_eachine>
+  </xacro:if>
   <gazebo reference="imu_link">
   </gazebo>

File: rosmip/rosmip_description/urdf/rosmip_1.urdf.xacro (robot description, xacro)
@@ -2,4 +2,5 @@
 <robot name="rosmip_1" xmlns:xacro="http://www.ros.org/wiki/xacro">
   <xacro:include filename="$(find rosmip_description)/urdf/rosmip_defaults.urdf.xacro" />
+  <xacro:property name="use_eachine_camera" value="true" />
   <xacro:include filename="$(find rosmip_description)/urdf/rosmip.urdf.xacro" />
 </robot>

File: rosmip/rosmip_description/urdf/rosmip_2.urdf.xacro (robot description, xacro)
@@ -2,7 +2,8 @@
 <robot name="rosmip_1" xmlns:xacro="http://www.ros.org/wiki/xacro">
   <xacro:include filename="$(find rosmip_description)/urdf/rosmip_defaults.urdf.xacro" />
-  <xacro:property name="left_wheel_radius"  value="0.045" />
-  <xacro:property name="right_wheel_radius" value="0.045" />
+  <xacro:property name="left_wheel_radius"  value="0.03" />
+  <xacro:property name="right_wheel_radius" value="0.03" />
   <xacro:property name="use_infrared_marker" value="true" />
+  <xacro:property name="use_eachine_camera" value="true" />
   <xacro:include filename="$(find rosmip_description)/urdf/rosmip.urdf.xacro" />
 </robot>

File: rosmip/rosmip_description/urdf/rosmip_defaults.urdf.xacro (robot description, xacro)
@@ -15,6 +15,8 @@
   <xacro:property name="high_definition_wheel_visual" value="true" />
   <xacro:property name="high_definition_body_visual"  value="true" />
+  <xacro:property name="high_definition_camera_visual"  value="true" />
   <!-- sensors -->
   <xacro:property name="use_infrared_marker" value="false" />
   <xacro:property name="use_aruco_marker"    value="false" />
+  <xacro:property name="use_eachine_camera" value="true" />
 </robot>

Commit message: added namespace to allow multi robot simulations

File: rosmip/rosmip_description/urdf/rosmip.urdf.xacro (robot description, xacro)
@@ -124,14 +124,7 @@
   <!-- Infrared Marker -->
   <xacro:if value="${use_infrared_marker}">
-     <xacro:arg name="root_link" default="irm_link"/>
-     <xacro:arg name="mesh" default="ir_marker.dae"/>
-     <xacro:include filename="$(find smocap)/urdf/ir_marker.urdf.xacro" />
-     <xacro:ir_marker root_link="$(arg root_link)" mesh="$(arg mesh)"/>
-    <xacro:property name="irm_z" value="0.12" />
-    <joint name="irm_joint" type="fixed">
-      <origin xyz="0 0 ${irm_z}" rpy="0 0 0" />
-      <parent link="chassis_link"/>
-      <child link="irm_link" />
-    </joint>
+    <xacro:cs_smocap_ir_marker mesh="${smocap_ir_marker_mesh}">
+      <origin xyz="0. 0. 0.092" rpy="0 0 0" />
+    </xacro:cs_smocap_ir_marker>
   </xacro:if>
   <!-- Aruco Marker -->

File: rosmip/rosmip_description/urdf/rosmip_1.urdf.xacro (robot description, xacro)
@@ -1,6 +1,9 @@
 <?xml version="1.0"?>
 <robot name="rosmip_1" xmlns:xacro="http://www.ros.org/wiki/xacro">
+  <xacro:arg name="robot_name" default="rosmip_1" />
   <xacro:include filename="$(find rosmip_description)/urdf/rosmip_defaults.urdf.xacro" />
-  <xacro:property name="use_eachine_camera" value="true" />
+  <xacro:property name="use_infrared_marker" value="true" />
+  <xacro:property name="smocap_ir_marker_mesh" value="ir_marker.dae" />
+  <xacro:property name="use_eachine_camera" value="false" />
   <xacro:include filename="$(find rosmip_description)/urdf/rosmip.urdf.xacro" />
 </robot>

File: rosmip/rosmip_description/urdf/rosmip_2.urdf.xacro (robot description, xacro)
@@ -1,9 +1,11 @@
 <?xml version="1.0"?>
 <robot name="rosmip_1" xmlns:xacro="http://www.ros.org/wiki/xacro">
+  <xacro:arg name="robot_name" default="rosmip_2" />
   <xacro:include filename="$(find rosmip_description)/urdf/rosmip_defaults.urdf.xacro" />
   <xacro:property name="left_wheel_radius"  value="0.03" />
   <xacro:property name="right_wheel_radius" value="0.03" />
   <xacro:property name="use_infrared_marker" value="true" />
-  <xacro:property name="use_eachine_camera" value="true" />
+  <xacro:property name="smocap_ir_marker_mesh" value="ir_marker_0.dae" />
+  <xacro:property name="use_eachine_camera" value="false" />
   <xacro:include filename="$(find rosmip_description)/urdf/rosmip.urdf.xacro" />
 </robot>

File: rosmip/rosmip_description/urdf/rosmip_defaults.urdf.xacro (robot description, xacro)
@@ -19,4 +19,4 @@
   <xacro:property name="use_infrared_marker" value="false" />
   <xacro:property name="use_aruco_marker"    value="false" />
-  <xacro:property name="use_eachine_camera" value="true" />
+  <xacro:property name="use_eachine_camera" value="false" />
 </robot>
